File: PCB/relay/v1.brd (EAGLE design)
At the start: 100 x 80 mm, 7 parts, among them T1 BC817, U1 SFH615A-07, U2 ALQ105

Commit message: Adding files for v0.2
Parts:
- R3: value 50k -> 10k
- moved U2 14.0 mm to (59.9, 30.4)
- moved R3 0.53 mm to (37.7, 23.9)
Connections:
- net 5V: now also U2.P$1; no longer U2.P$2
- net N$4: now also U2.P$2; no longer U2.P$1
Routing:
- net N$4: track 7.85 -> 12.4 mm
- net 5V: track 8.70 -> 13.3 mm
- net N$3: track 4.37 -> 4.90 mm
Changed lines of the file:
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@@
 <attribute name="NAME" x="36.6014" y="28.7528" size="1.27" layer="25" font="vector" rot="R180"/>
 </element>
-<element name="R3" library="SparkFun-Passives" package="0603-RES" value="50k" x="37.7444" y="24.4602" smashed="yes" rot="R90">
-<attribute name="NAME" x="36.6268" y="24.9428" size="1.27" layer="25" font="vector" rot="R180"/>
-</element>
-<element name="T1" library="lib" package="BC817" value="BC817" x="41.021" y="26.67" smashed="yes" rot="R270">
+<element name="T1" library="lib" library_urn="urn:adsk.eagle:library:473707" package="BC817" package3d_urn="urn:adsk.eagle:package:473719/1" value="BC817" x="41.021" y="26.67" smashed="yes" rot="R270">
 <attribute name="NAME" x="40.2004" y="23.8742" size="1.27" layer="25"/>
 </element>
-<element name="U1" library="lib" package="SFH615A-07" value="SFH615A-07" x="33.02" y="33.02" smashed="yes">
+<element name="U1" library="lib" library_urn="urn:adsk.eagle:library:473707" package="SFH615A-07" package3d_urn="urn:adsk.eagle:package:473718/1" value="SFH615A-07" x="33.02" y="33.02" smashed="yes">
 <attribute name="NAME" x="29.74" y="36.23" size="1.27" layer="25"/>
 </element>
-<element name="U2" library="lib" package="ALQ105" value="ALQ105" x="46.482" y="26.67" smashed="yes">
-<attribute name="NAME" x="46.1772" y="36.576" size="1.27" layer="21"/>
+<element name="U2" library="lib" library_urn="urn:adsk.eagle:library:473707" package="ALQ105" package3d_urn="urn:adsk.eagle:package:473720/1" value="ALQ105" x="59.944" y="30.4292" smashed="yes">
+<attribute name="NAME" x="59.6392" y="40.3352" size="1.27" layer="21"/>
 </element>
+<element name="R3" library="SparkFun-Passives" package="0603-RES" value="10k" x="37.7444" y="23.9268" rot="R90"/>
 </elements>
 <signals>
@@
 <signal name="GND">
 <contactref element="U1" pad="P$2"/>
+<contactref element="T1" pad="P$3"/>
 <contactref element="R3" pad="1"/>
-<contactref element="T1" pad="P$3"/>
-<wire x1="40.071" y1="26.02" x2="28.255" y2="31.75" width="0" layer="19" extent="1-1"/>
-<wire x1="37.7444" y1="23.6102" x2="40.071" y2="26.02" width="0" layer="19" extent="1-1"/>
+<wire x1="28.255" y1="31.75" x2="40.071" y2="26.02" width="0" layer="19" extent="1-1"/>
+<wire x1="37.7444" y1="23.0768" x2="28.255" y2="31.75" width="0" layer="19" extent="1-1"/>
 </signal>
 <signal name="N$2">
@@
 <signal name="N$3">
 <contactref element="R2" pad="1"/>
-<contactref element="R3" pad="2"/>
 <contactref element="T1" pad="P$2"/>
 <wire x1="37.7952" y1="27.32" x2="40.071" y2="27.32" width="0.4064" layer="1"/>
 <wire x1="37.7952" y1="27.32" x2="37.7684" y2="27.32" width="0.4064" layer="1"/>
 <wire x1="37.7684" y1="27.32" x2="37.7444" y2="27.344" width="0.4064" layer="1"/>
-<wire x1="37.7444" y1="25.3102" x2="37.7444" y2="27.2692" width="0.4064" layer="1"/>
-<wire x1="37.7444" y1="27.2692" x2="37.7952" y2="27.32" width="0.4064" layer="1"/>
+<wire x1="37.7952" y1="27.32" x2="37.7444" y2="27.2692" width="0.4064" layer="1"/>
+<contactref element="R3" pad="2"/>
+<wire x1="37.7444" y1="27.2692" x2="37.7444" y2="24.7768" width="0.4064" layer="1"/>
 </signal>
 <signal name="5V">
 <contactref element="U1" pad="P$4"/>
 <contactref element="D1" pad="C"/>
-<contactref element="U2" pad="P$2"/>
 <wire x1="37.785" y1="34.29" x2="41.901" y2="34.29" width="0.4064" layer="1"/>
 <wire x1="41.901" y1="34.29" x2="41.91" y2="34.281" width="0.4064" layer="1"/>
-<wire x1="41.91" y1="34.281" x2="46.473" y2="34.281" width="0.4064" layer="1"/>
-<wire x1="46.473" y1="34.281" x2="46.482" y2="34.29" width="0.4064" layer="1"/>
+<contactref element="U2" pad="P$1"/>
+<wire x1="51.0122" y1="34.281" x2="51.054" y2="34.2392" width="0.4064" layer="1"/>
+<wire x1="41.91" y1="34.281" x2="51.0122" y2="34.281" width="0.4064" layer="1"/>
 </signal>
 <signal name="N$4">
 <contactref element="D1" pad="A"/>
 <contactref element="T1" pad="P$1"/>
-<contactref element="U2" pad="P$1"/>
 <wire x1="41.91" y1="29.981" x2="41.91" y2="26.731" width="0.4064" layer="1"/>
-<wire x1="41.971" y1="26.67" x2="41.91" y2="26.731" width="0.4064" layer="1"/>
-<wire x1="46.482" y1="26.67" x2="41.971" y2="26.67" width="0.4064" layer="1"/>
+<wire x1="41.91" y1="26.731" x2="41.971" y2="26.67" width="0.4064" layer="1"/>
+<contactref element="U2" pad="P$2"/>
+<wire x1="41.971" y1="26.67" x2="51.0032" y2="26.67" width="0.4064" layer="1"/>
+<wire x1="51.0032" y1="26.67" x2="51.054" y2="26.6192" width="0.4064" layer="1"/>
 </signal>
 </signals>
 </board>
 </drawing>
+<compatibility>
+<note version="8.2" severity="warning">
+Since Version 8.2, EAGLE supports online libraries. The ids
+of those online libraries will not be understood (or retained)
+with this version.
+</note>
+<note version="8.3" severity="warning">
+Since Version 8.3, EAGLE supports URNs for individual library
+assets (packages, symbols, and devices). The URNs of those assets
+will not be understood (or retained) with this version.
+</note>
+<note version="8.3" severity="warning">
+Since Version 8.3, EAGLE supports the association of 3D packages
+with devices in libraries, schematics, and board files. Those 3D
+packages will not be understood (or retained) with this version.
+</note>
+</compatibility>
 </eagle>

Commit message: Adding files
Parts:
- moved R2 0.15 mm to (37.7, 28.3)
Routing:
- net N$3: track 4.90 -> 5.71 mm
Changed lines of the file:
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@@
 <?xml version="1.0" encoding="utf-8"?>
 <!DOCTYPE eagle SYSTEM "eagle.dtd">
-<eagle version="8.3.2">
+<eagle version="8.4.3">
 <drawing>
 <settings>
@@
 <param name="dpMaxLengthDifference" value="10mm"/>
 <param name="dpGapFactor" value="2.5"/>
-<param name="checkGrid" value="0"/>
 <param name="checkAngle" value="0"/>
 <param name="checkFont" value="1"/>
 <param name="checkRestrict" value="1"/>
+<param name="checkStop" value="0"/>
 <param name="useDiameter" value="13"/>
 <param name="maxErrors" value="50"/>
@@
 <attribute name="VALUE" x="40.259" y="32.385" size="0.4064" layer="27" rot="R90"/>
 </element>
-<element name="R1" library="SparkFun-Passives" package="0603-RES" value="50" x="24.13" y="34.29"/>
-<element name="R2" library="SparkFun-Passives" package="0603-RES" value="10k" x="37.7444" y="28.194" smashed="yes" rot="R90">
-<attribute name="NAME" x="36.6014" y="28.7528" size="1.27" layer="25" font="vector" rot="R180"/>
+<element name="R1" library="SparkFun-Passives" package="0603-RES" value="50" x="24.13" y="34.29" smashed="yes">
+<attribute name="NAME" x="23.241" y="35.9664" size="1.27" layer="25"/>
+</element>
+<element name="R2" library="SparkFun-Passives" package="0603-RES" value="10k" x="37.7444" y="28.3464" smashed="yes" rot="R90">
+<attribute name="NAME" x="36.6014" y="28.194" size="1.27" layer="25" font="vector" rot="R180"/>
 </element>
 <element name="T1" library="lib" library_urn="urn:adsk.eagle:library:473707" package="BC817" package3d_urn="urn:adsk.eagle:package:473719/1" value="BC817" x="41.021" y="26.67" smashed="yes" rot="R270">
-<attribute name="NAME" x="40.2004" y="23.8742" size="1.27" layer="25"/>
+<attribute name="NAME" x="40.048" y="23.2138" size="1.27" layer="25"/>
 </element>
 <element name="U1" library="lib" library_urn="urn:adsk.eagle:library:473707" package="SFH615A-07" package3d_urn="urn:adsk.eagle:package:473718/1" value="SFH615A-07" x="33.02" y="33.02" smashed="yes">
-<attribute name="NAME" x="29.74" y="36.23" size="1.27" layer="25"/>
+<attribute name="NAME" x="29.8924" y="36.2808" size="1.27" layer="25"/>
 </element>
 <element name="U2" library="lib" library_urn="urn:adsk.eagle:library:473707" package="ALQ105" package3d_urn="urn:adsk.eagle:package:473720/1" value="ALQ105" x="59.944" y="30.4292" smashed="yes">
-<attribute name="NAME" x="59.6392" y="40.3352" size="1.27" layer="21"/>
-</element>
-<element name="R3" library="SparkFun-Passives" package="0603-RES" value="10k" x="37.7444" y="23.9268" rot="R90"/>
+<attribute name="NAME" x="49.9364" y="36.2712" size="1.27" layer="21"/>
+</element>
+<element name="R3" library="SparkFun-Passives" package="0603-RES" value="10k" x="37.7444" y="23.9268" smashed="yes" rot="R90">
+<attribute name="NAME" x="36.6522" y="23.7744" size="1.27" layer="25" rot="R180"/>
+<attribute name="VALUE" x="38.8874" y="22.9108" size="0.4064" layer="27" font="vector" rot="R90"/>
+</element>
 </elements>
 <signals>
@@
 <contactref element="T1" pad="P$3"/>
 <contactref element="R3" pad="1"/>
-<wire x1="28.255" y1="31.75" x2="40.071" y2="26.02" width="0" layer="19" extent="1-1"/>
+<wire x1="28.255" y1="31.75" x2="40.0252" y2="25.645" width="0" layer="19" extent="1-1"/>
 <wire x1="37.7444" y1="23.0768" x2="28.255" y2="31.75" width="0" layer="19" extent="1-1"/>
 </signal>
@@
 <contactref element="R2" pad="2"/>
 <wire x1="37.785" y1="31.75" x2="37.785" y2="29.0846" width="0.4064" layer="1"/>
-<wire x1="37.785" y1="29.0846" x2="37.7444" y2="29.044" width="0.4064" layer="1"/>
+<wire x1="37.785" y1="29.0846" x2="37.7444" y2="29.1964" width="0.4064" layer="1"/>
 </signal>
 <signal name="N$3">
 <contactref element="R2" pad="1"/>
 <contactref element="T1" pad="P$2"/>
-<wire x1="37.7952" y1="27.32" x2="40.071" y2="27.32" width="0.4064" layer="1"/>
-<wire x1="37.7952" y1="27.32" x2="37.7684" y2="27.32" width="0.4064" layer="1"/>
-<wire x1="37.7684" y1="27.32" x2="37.7444" y2="27.344" width="0.4064" layer="1"/>
-<wire x1="37.7952" y1="27.32" x2="37.7444" y2="27.2692" width="0.4064" layer="1"/>
+<wire x1="37.7444" y1="27.6756" x2="40.0252" y2="27.695" width="0.4064" layer="1"/>
+<wire x1="37.7444" y1="27.6756" x2="37.7684" y2="27.32" width="0.4064" layer="1"/>
+<wire x1="37.7684" y1="27.32" x2="37.7444" y2="27.4964" width="0.4064" layer="1"/>
 <contactref element="R3" pad="2"/>
-<wire x1="37.7444" y1="27.2692" x2="37.7444" y2="24.7768" width="0.4064" layer="1"/>
+<wire x1="37.7444" y1="27.6756" x2="37.7444" y2="24.7768" width="0.4064" layer="1"/>
 </signal>
 <signal name="5V">
@@
 <contactref element="T1" pad="P$1"/>
 <wire x1="41.91" y1="29.981" x2="41.91" y2="26.731" width="0.4064" layer="1"/>
-<wire x1="41.91" y1="26.731" x2="41.971" y2="26.67" width="0.4064" layer="1"/>
+<wire x1="41.91" y1="26.731" x2="42.0168" y2="26.67" width="0.4064" layer="1"/>
 <contactref element="U2" pad="P$2"/>
-<wire x1="41.971" y1="26.67" x2="51.0032" y2="26.67" width="0.4064" layer="1"/>
+<wire x1="42.0168" y1="26.67" x2="51.0032" y2="26.67" width="0.4064" layer="1"/>
 <wire x1="51.0032" y1="26.67" x2="51.054" y2="26.6192" width="0.4064" layer="1"/>
 </signal>
