File: PCB/mainPCB/mainPCB.sch (EAGLE design)
At the start: 58 parts, among them CN1 SDS-50J, CN2 SDS-50J, CN3 SDS-50J, CN4 SDS-50J, J2 RASPBERRYPI-40-PIN-GPIO, T2 BC817, T3 BC817, T4 BC817, T6 BC817, U1 AT24C256C-SSHL-B, U11 SFH615A-07, U12 ALQ105, U3 SFH615A-07, U4 ALQ105, U5 SFH615A-07, U6 ALQ105, U7 SFH615A-07, U8 ALQ105

Commit message: Adding files for v0.2
Parts:
- removed J1, J3, J4, J5: (no value), SparkFun-Connectors:M022.54MM_SCREWTERM
- removed U$1: MCP3208I/SL, adcLib:MCP3208I/SL
- added C10, C11, C2, C3, C4, C5, C6, C7, C8, C9: 0.1uF, SparkFun-Capacitors:0.1UF-25V(+80/-20%)(0603)
- added C12, C13: 10uF, SparkFun-Capacitors:1.0UF50V10%(1206)
- added C14, C15: EEE-HA1C471UPCAP_PAN_EEE_F-L, EEE-HA1C471UP:EEE-HA1C471UPCAP_PAN_EEE_F-L
- added CN5, CN6, CN7, CN8: SDS-50J, SDS-50J:SDS-50J
- added CON1: 1776244-4, lib:1776244-4
- added D10, D11, D5, D8, D9: (no value), SparkFun-DiscreteSemi:DIODESMA
- added F5, F6, F7, F8: 3544-2, lib:3544-2
- added FRAME3: FRAME-LETTER, SparkFun-Aesthetics:FRAME-LETTER
- added Q1: DMMT5401-7-F, DMMT5401-7-F:DMMT5401-7-F
- added R24: 0, SparkFun-Passives:RESISTOR1206
- added R25, R40, R43, R46, R49: 10k, SparkFun-Passives:RESISTOR0603-RES
- added R26, R41, R44, R47, R50: 47k, SparkFun-Passives:RESISTOR0603-RES
- added R27: DNP, SparkFun-Passives:RESISTOR1206
- added R28, R29, R30, R31, R32, R33, R34, R35: 330, SparkFun-Passives:RESISTOR0603-RES
- added R39, R42, R45, R48: 47, SparkFun-Passives:RESISTOR0603-RES
- added T5, T7, T8, T9: BC817, lib:BC817
- added U$2: MCP3208T-CI/SL, MCP3208T-CI_SL:MCP3208T-CI/SL
- added U13, U15, U17, U19: SFH615A-07, lib:SFH615A-07
- added U14, U16, U18, U20: ALQ105, lib:ALQ105
- added U2: DMG2305UX-13SOT-23-M, DMG2359UX:DMG2305UX-13SOT-23-M
- R14, R15: device SparkFun-Passives:RESISTOR0603-RES -> SparkFun-Passives:RESISTOR1206
- R21: value 1k -> 3.9k
Connections:
- new net 5V_RPI: C12.1, C13.1, Q1.E1, R14.1, R27.1, U2.D
- new net A1_F: C2.1, CN1.2, R28.2
- new net A2_F: C3.1, CN2.2, R29.2
- new net A3_F: C4.1, CN3.2, R30.2
- new net A4_F: C5.1, CN4.2, R31.2
- new net A5_F: C6.1, CN5.2, R32.2
- new net A6_F: C7.1, CN6.2, R33.2
- new net A7_F: C8.1, CN7.2, R34.2
- new net A8_F: C9.1, CN8.2, R35.2
- new net N$29: Q1.C2, R26.2, U2.G
- new net N$30: CON1.PIN4, D5.A
- new net N$31: F5.P$1, U14.COM
- new net N$32: F6.P$1, U16.COM
- new net N$33: F7.P$1, U20.COM
- new net N$34: F8.P$1, U18.COM
- new net N$35: R39.2, U13.LED+
- new net N$36: C10.1, C11.1, R19.1, U$2.VDD, U$2.VREF
- new net N$37: R40.2, U13.OUT-
- new net N$38: R40.1, R41.2, T5.B
- new net N$39: D8.A, T5.C, U14.COM+
- new net N$40: R42.2, U15.LED+
- new net N$41: R43.2, U15.OUT-
- new net N$42: R43.1, R44.2, T7.B
- new net N$43: D9.A, T7.C, U16.COM+
- new net N$44: R45.2, U17.LED+
- new net N$45: R46.2, U17.OUT-
- new net N$46: R46.1, R47.2, T8.B
- new net N$47: D10.A, T8.C, U18.COM+
- new net N$48: R48.2, U19.LED+
- new net N$49: R49.2, U19.OUT-
- new net N$50: R49.1, R50.2, T9.B
- new net N$51: D11.A, T9.C, U20.COM+
- new net R5: CN5.5, U14.NO
- new net R6: CN6.5, U16.NO
- new net R7: CN7.5, U20.NO
- new net R8: CN8.5, U18.NO
- new net RELAY5: J2.GP27, R39.1
- new net RELAY6: J2.GP22, R42.1
- new net RELAY7: J2.GP5, R48.1
- new net RELAY8: J2.GP6, R45.1
- net 12V: now also D5.C, F5.P$2, F6.P$2, F7.P$2, F8.P$2; no longer J4.1, J4.2
- net 3_3V: no longer J1.1, J1.2, U$1.VREF
- net 5V: now also C14.11, C15.11, CN5.1, CN6.1, CN7.1, CN8.1, CON1.PIN1, D10.C, D11.C, D8.C, D9.C, Q1.E2, R27.2, U12.COM-, U13.OUT+, U14.COM-, U15.OUT+, U16.COM-, U17.OUT+, U18.COM-, U19.OUT+, U2.S, U20.COM-, U4.COM-, U6.COM-, U8.COM-; no longer J3.1, J3.2, R14.1, U12.COM+, U4.COM+, U6.COM+, U8.COM+
- net A1: now also R28.1, U$2.CH0; no longer CN1.2, U$1.CH0
- net A2: now also R29.1, U$2.CH1; no longer CN2.2, U$1.CH1
- net A3: now also R30.1, U$2.CH2; no longer CN3.2, U$1.CH2
- net A4: now also R31.1, U$2.CH3; no longer CN4.2, U$1.CH3
- net A5: now also R32.1, U$2.CH4; no longer U$1.CH4
- net A6: now also R33.1, U$2.CH5; no longer U$1.CH5
- net A7: now also R34.1, U$2.CH6; no longer U$1.CH6
- net A8: now also R35.1, U$2.CH7; no longer U$1.CH7
- net AGND: now also U$2.AGND; no longer U$1.AGND
- net CLK: now also U$2.CLK; no longer U$1.CLK
- net COM: now also CN5.3, CN6.3, CN7.3, CN8.3, R24.1
- net CS_ADC: now also U$2.*CS/SHDN; no longer U$1.!CS
- net GND: now also C10.2, C11.2, C12.2, C13.2, C14.22, C15.22, C2.2, C3.2, C4.2, C5.2, C6.2, C7.2, C8.2, C9.2, CN5.4, CN6.4, CN7.4, CN8.4, CON1.PIN2, CON1.PIN3, R24.2, R25.1, R26.1, R41.1, R44.1, R47.1, R50.1, T5.E, T7.E, T8.E, T9.E, U$2.DGND, U13.LED-, U15.LED-, U17.LED-, U19.LED-; no longer J5.1, J5.2, U$1.DGND
- net MISO: now also U$2.DOUT; no longer U$1.DOUT
- net MOSI: now also U$2.DIN; no longer U$1.DIN
- net N$12: now also U6.COM+; no longer U6.COM-
- net N$16: now also U8.COM+; no longer U8.COM-
- net N$24: now also U12.COM+; no longer U12.COM-
- net N$27: now also Q1.B1, Q1.B2, Q1.C1, R25.2; no longer R19.1, U$1.VDD
- net N$8: now also U4.COM+; no longer U4.COM-
Other:
- note added: "Still to do... - Caps - Verify ADC w/ flow sensor"
- note added: "Update Footprint!"

Commit message: Removed Diode.
Parts:
- removed D5: (no value), SparkFun-DiscreteSemi:DIODESMA
Connections:
- removed net N$30: CON1.PIN4, D5.A
- net 12V: now also CON1.PIN4; no longer D5.C
Other:
- note added: "Fuse"
- note added: "G5Q"
- note added: "Protection: - in front of ADC (TVS) - on 12V Line @ fuse (TVS) - Fuse on 12V line"
- note added: "TVS Diode"
- note removed: "Still to do... - Caps - Verify ADC w/ flow sensor"
- note removed: "Update Footprint!"
Changed lines of the file:
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@@
 <?xml version="1.0" encoding="utf-8"?>
 <!DOCTYPE eagle SYSTEM "eagle.dtd">
-<eagle version="8.4.3">
+<eagle version="8.3.2">
 <drawing>
 <settings>
@@
 <part name="C8" library="SparkFun-Capacitors" deviceset="0.1UF-25V(+80/-20%)(0603)" device="" value="0.1uF"/>
 <part name="C9" library="SparkFun-Capacitors" deviceset="0.1UF-25V(+80/-20%)(0603)" device="" value="0.1uF"/>
-<part name="D5" library="SparkFun-DiscreteSemi" deviceset="DIODE" device="SMA"/>
 <part name="FRAME3" library="SparkFun-Aesthetics" deviceset="FRAME-LETTER" device=""/>
 <part name="U13" library="lib" deviceset="SFH615A-07" device=""/>
@@
 <plain>
 <text x="190.5" y="78.74" size="1.778" layer="91">Recommended: CAT24C256WI-GT3</text>
-<text x="185.42" y="203.2" size="1.778" layer="91">RPi Recommendations (Power):
+<text x="167.64" y="175.26" size="1.778" layer="91">RPi Recommendations (Power):
 https://github.com/raspberrypi/hats/blob/master/designguide.md</text>
-<text x="104.14" y="193.04" size="1.778" layer="91">Still to do...
-- Caps
-- Verify ADC w/ flow sensor
-</text>
+<text x="101.6" y="40.64" size="1.778" layer="91">G5Q </text>
+<text x="81.28" y="12.7" size="1.778" layer="91">Fuse</text>
+<text x="139.7" y="81.28" size="1.778" layer="91">Protection:
+- in front of ADC (TVS)
+- on 12V Line @ fuse (TVS)
+- Fuse on 12V line</text>
 </plain>
 <instances>
@@
 <instance part="C8" gate="G$1" x="33.02" y="40.64"/>
 <instance part="C9" gate="G$1" x="33.02" y="17.78"/>
-<instance part="D5" gate="G$1" x="83.82" y="17.78"/>
 <instance part="C10" gate="G$1" x="147.32" y="154.94"/>
 <instance part="C11" gate="G$1" x="132.08" y="154.94"/>
@@
 </segment>
 </net>
-<net name="N$30" class="0">
-<segment>
+<net name="12V" class="0">
+<segment>
+<label x="93.98" y="17.78" size="1.778" layer="95"/>
 <pinref part="CON1" gate="A" pin="PIN4"/>
-<pinref part="D5" gate="G$1" pin="A"/>
-<wire x1="73.66" y1="17.78" x2="81.28" y2="17.78" width="0.1524" layer="91"/>
-</segment>
-</net>
-<net name="12V" class="0">
-<segment>
-<pinref part="D5" gate="G$1" pin="C"/>
-<wire x1="86.36" y1="17.78" x2="93.98" y2="17.78" width="0.1524" layer="91"/>
-<label x="93.98" y="17.78" size="1.778" layer="95"/>
+<wire x1="73.66" y1="17.78" x2="93.98" y2="17.78" width="0.1524" layer="91"/>
 </segment>
 </net>
@@
 <description>Relays 1-2</description>
 <plain>
-<text x="96.52" y="129.54" size="1.778" layer="91">Update Footprint!</text>
+<text x="119.38" y="170.18" size="1.778" layer="91">TVS Diode</text>
 </plain>
 <instances>

Commit message: Technically version 0.4. Sending it to JLCPCB for production.
Parts:
- removed CON1: 1776244-4, lib:1776244-4
- added D1, D12, D13, D14, D15, D16, D5, D7: BAV99-7-F, SparkFun-DiscreteSemi:BAV99
- added F9: 3544-2, lib:3544-2
- added J1: 1935161, 1935161:1935161
- added L1: DR73-1R0-R, DR73-1R0-R:DR73-1R0-R
- added R36: 0, SparkFun-Passives:RESISTOR1206
- added TP_ON/OFF, TP_TRIM: TEST-POINT3X5, SparkFun-Passives:TEST-POINT3X5
- added U9: S24SE05004PDFA, S24SE05004PDFA:S24SE05004PDFA
- C1, C10, C11, C14, C15, C2, C3, C4, C5, C6, C7, C8, C9, CN1, CN2, CN3, CN4, CN5, CN6, CN7, CN8, D10, D11, D2, D3, D4, D6, D8, D9, F1, F2, F3, F4, F5, F6, F7, F8, J2, J6, Q1, R1, R10, R11, R12, R13, R14, R15, R16, R17, R18, R19, R2, R20, R21, R22, R23, R24, R25, R26, R28, R29, R3, R30, R31, R32, R33, R34, R35, R39, R4, R40, R41, R42, R43, R44, R45, R46, R47, R48, R49, R5, R50, R6, R7, R8, R9, T2, T3, T4, T5, T6, T7, T8, T9, U$2, U1, U11, U12, U13, U14, U15, U16, U17, U18, U19, U2, U20, U3, U4, U5, U6, U7, U8: POPULATE (none) -> Y
- C12, C13: value 10uF -> 1uF; POPULATE (none) -> Y
- FRAME1, FRAME2, FRAME3, R27: POPULATE (none) -> N
Connections:
- new net N$30: TP_ON/OFF.1, U9.ON/OFF
- new net N$52: L1.1, U9.VIN+
- new net N$53: TP_TRIM.1, U9.TRIM
- new net N$54: F9.P$1, J1.1
- net 12V: now also C14.11, C15.11, F9.P$2, L1.2; no longer CON1.PIN4
- net 5V: now also D1.C2, D12.C2, D13.C2, D14.C2, D15.C2, D16.C2, D5.C2, D7.C2, Q1.E1, R27.1, U2.D, U9.VOUT+; no longer C14.11, C15.11, CON1.PIN1, Q1.E2, R27.2, U2.S
- net 5V_RPI: now also Q1.E2, R27.2, U2.S; no longer Q1.E1, R27.1, U2.D
- net A1_F: now also D1.COM
- net A2_F: now also D5.COM
- net A3_F: now also D7.COM
- net A4_F: now also D12.COM
- net A5_F: now also D13.COM
- net A6_F: now also D14.COM
- net A7_F: now also D15.COM
- net A8_F: now also D16.COM
- net COM: now also R36.1
- net GND: now also D1.A1, D12.A1, D13.A1, D14.A1, D15.A1, D16.A1, D5.A1, D7.A1, J1.2, R36.2, U9.VIN-, U9.VOUT-; no longer CON1.PIN2, CON1.PIN3
Other:
- note added: "Leave ON/OFF floating for P version"
- note added: "Possible relay replacement G5Q"
- note removed: "Fuse"
- note removed: "G5Q"
- note removed: "Protection: - in front of ADC (TVS) - on 12V Line @ fuse (TVS) - Fuse on 12V line"
- moved on the sheet: C10, C11, C12, C13, C14, C15, J2, Q1, R1, R13, R14, R15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

Commit message: Added all design files for v0.4. Cleaned up old files.
Other:
- note removed: "TVS Diode"
- moved on the sheet: C14, C15, L1, TP_ON/OFF, TP_TRIM, U9
Changed lines of the file:
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@@
 <?xml version="1.0" encoding="utf-8"?>
 <!DOCTYPE eagle SYSTEM "eagle.dtd">
-<eagle version="8.6.3">
+<eagle version="8.6.0">
 <drawing>
 <settings>
@@
 https://github.com/raspberrypi/hats/blob/master/designguide.md</text>
 <text x="185.42" y="175.26" size="1.778" layer="97">Possible relay replacement G5Q</text>
-<text x="259.08" y="119.38" size="1.778" layer="97">Leave ON/OFF floating for P version</text>
+<text x="256.54" y="60.96" size="1.778" layer="97" rot="R90">Leave ON/OFF floating for P version</text>
 </plain>
 <instances>
@@
 <attribute name="POPULATE" x="175.26" y="129.54" size="1.778" layer="96" display="off"/>
 </instance>
-<instance part="C14" gate="A" x="330.2" y="106.68" smashed="yes" rot="R270">
-<attribute name="NAME" x="331.1906" y="106.2228" size="1.778" layer="95" ratio="10" rot="SR0"/>
-<attribute name="POPULATE" x="330.2" y="106.68" size="1.778" layer="96" rot="R270" display="off"/>
-</instance>
-<instance part="C15" gate="A" x="342.9" y="106.68" smashed="yes" rot="R270">
-<attribute name="NAME" x="343.8906" y="106.2228" size="1.778" layer="95" ratio="10" rot="SR0"/>
-<attribute name="POPULATE" x="342.9" y="106.68" size="1.778" layer="96" rot="R270" display="off"/>
+<instance part="C14" gate="A" x="269.24" y="132.08" smashed="yes">
+<attribute name="NAME" x="269.6972" y="133.0706" size="1.778" layer="95" ratio="10" rot="SR90"/>
+<attribute name="POPULATE" x="269.24" y="132.08" size="1.778" layer="96" display="off"/>
+</instance>
+<instance part="C15" gate="A" x="269.24" y="144.78" smashed="yes">
+<attribute name="NAME" x="269.6972" y="145.7706" size="1.778" layer="95" ratio="10" rot="SR90"/>
+<attribute name="POPULATE" x="269.24" y="144.78" size="1.778" layer="96" display="off"/>
 </instance>
 <instance part="D1" gate="G$1" x="60.96" y="177.8">
@@
 <attribute name="POPULATE" x="101.6" y="15.24" size="1.778" layer="96" display="off"/>
 </instance>
-<instance part="L1" gate="A" x="320.04" y="111.76" smashed="yes" rot="R90">
-<attribute name="VALUE" x="314.96" y="117.9322" size="1.778" layer="96" ratio="10" rot="SR180" align="bottom-right"/>
-<attribute name="NAME" x="314.96" y="119.8372" size="1.778" layer="95" ratio="10" rot="SR180" align="bottom-right"/>
-</instance>
-<instance part="U9" gate="G$1" x="279.4" y="104.14" rot="MR0"/>
-<instance part="TP_ON/OFF" gate="G$1" x="307.34" y="88.9" smashed="yes">
-<attribute name="NAME" x="307.34" y="86.36" size="1.778" layer="95"/>
-</instance>
-<instance part="TP_TRIM" gate="G$1" x="304.8" y="83.82" smashed="yes">
-<attribute name="NAME" x="304.8" y="81.28" size="1.778" layer="95"/>
+<instance part="L1" gate="A" x="264.16" y="121.92" smashed="yes" rot="R180">
+<attribute name="VALUE" x="257.9878" y="116.84" size="1.778" layer="96" ratio="10" rot="SR270" align="bottom-right"/>
+<attribute name="NAME" x="256.0828" y="116.84" size="1.778" layer="95" ratio="10" rot="SR270" align="bottom-right"/>
+</instance>
+<instance part="U9" gate="G$1" x="271.78" y="81.28" rot="MR270"/>
+<instance part="TP_ON/OFF" gate="G$1" x="287.02" y="109.22" smashed="yes" rot="R90">
+<attribute name="NAME" x="289.56" y="109.22" size="1.778" layer="95" rot="R90"/>
+</instance>
+<instance part="TP_TRIM" gate="G$1" x="292.1" y="106.68" smashed="yes" rot="R90">
+<attribute name="NAME" x="294.64" y="106.68" size="1.778" layer="95" rot="R90"/>
 </instance>
 <instance part="J1" gate="G$1" x="86.36" y="17.78" smashed="yes" rot="R180">
@@
 <segment>
 <pinref part="C14" gate="A" pin="22"/>
-<wire x1="330.2" y1="99.06" x2="330.2" y2="96.52" width="0.1524" layer="91"/>
-<label x="327.66" y="93.98" size="1.778" layer="95"/>
+<wire x1="276.86" y1="132.08" x2="279.4" y2="132.08" width="0.1524" layer="91"/>
+<label x="281.94" y="129.54" size="1.778" layer="95" rot="R90"/>
 </segment>
 <segment>
 <pinref part="C15" gate="A" pin="22"/>
-<wire x1="342.9" y1="99.06" x2="342.9" y2="96.52" width="0.1524" layer="91"/>
-<label x="340.36" y="93.98" size="1.778" layer="95"/>
+<wire x1="276.86" y1="144.78" x2="279.4" y2="144.78" width="0.1524" layer="91"/>
+<label x="281.94" y="142.24" size="1.778" layer="95" rot="R90"/>
 </segment>
 <segment>
@@
 <segment>
 <pinref part="U9" gate="G$1" pin="VIN-"/>
-<wire x1="302.26" y1="106.68" x2="312.42" y2="106.68" width="0.1524" layer="91"/>
-<wire x1="312.42" y1="106.68" x2="312.42" y2="96.52" width="0.1524" layer="91"/>
-<label x="309.88" y="93.98" size="1.778" layer="95"/>
+<wire x1="269.24" y1="104.14" x2="269.24" y2="114.3" width="0.1524" layer="91"/>
+<wire x1="269.24" y1="114.3" x2="279.4" y2="114.3" width="0.1524" layer="91"/>
+<label x="281.94" y="111.76" size="1.778" layer="95" rot="R90"/>
 </segment>
 <segment>
 <pinref part="U9" gate="G$1" pin="VOUT-"/>
-<wire x1="256.54" y1="106.68" x2="254" y2="106.68" width="0.1524" layer="91"/>
-<wire x1="254" y1="106.68" x2="254" y2="96.52" width="0.1524" layer="91"/>
-<label x="251.46" y="93.98" size="1.778" layer="95"/>
+<wire x1="269.24" y1="58.42" x2="269.24" y2="55.88" width="0.1524" layer="91"/>
+<wire x1="269.24" y1="55.88" x2="279.4" y2="55.88" width="0.1524" layer="91"/>
+<label x="281.94" y="53.34" size="1.778" layer="95" rot="R90"/>
 </segment>
 <segment>
@@
 <segment>
 <pinref part="U9" gate="G$1" pin="VOUT+"/>
-<wire x1="256.54" y1="109.22" x2="254" y2="109.22" width="0.1524" layer="91"/>
-<label x="254" y="109.22" size="1.778" layer="95" rot="MR0"/>
+<wire x1="266.7" y1="58.42" x2="266.7" y2="55.88" width="0.1524" layer="91"/>
+<label x="266.7" y="55.88" size="1.778" layer="95" rot="MR270"/>
 </segment>
 </net>
@@
 <segment>
 <pinref part="L1" gate="A" pin="2"/>
-<wire x1="342.9" y1="109.22" x2="330.2" y2="109.22" width="0.1524" layer="91"/>
+<wire x1="266.7" y1="144.78" x2="266.7" y2="132.08" width="0.1524" layer="91"/>
 <pinref part="C15" gate="A" pin="11"/>
-<wire x1="330.2" y1="109.22" x2="325.12" y2="109.22" width="0.1524" layer="91"/>
-<wire x1="342.9" y1="106.68" x2="342.9" y2="109.22" width="0.1524" layer="91"/>
+<wire x1="266.7" y1="132.08" x2="266.7" y2="127" width="0.1524" layer="91"/>
+<wire x1="269.24" y1="144.78" x2="266.7" y2="144.78" width="0.1524" layer="91"/>
 <pinref part="C14" gate="A" pin="11"/>
-<wire x1="330.2" y1="106.68" x2="330.2" y2="109.22" width="0.1524" layer="91"/>
-<junction x="330.2" y="109.22"/>
-<label x="335.28" y="109.22" size="1.778" layer="95"/>
+<wire x1="269.24" y1="132.08" x2="266.7" y2="132.08" width="0.1524" layer="91"/>
+<junction x="266.7" y="132.08"/>
+<label x="266.7" y="137.16" size="1.778" layer="95" rot="R90"/>
 </segment>
 </net>
@@
 <pinref part="L1" gate="A" pin="1"/>
 <pinref part="U9" gate="G$1" pin="VIN+"/>
-<wire x1="314.96" y1="109.22" x2="302.26" y2="109.22" width="0.1524" layer="91"/>
+<wire x1="266.7" y1="116.84" x2="266.7" y2="104.14" width="0.1524" layer="91"/>
 </segment>
 </net>
@@
 <segment>
 <pinref part="U9" gate="G$1" pin="ON/OFF"/>
-<wire x1="302.26" y1="101.6" x2="307.34" y2="101.6" width="0.1524" layer="91"/>
-<wire x1="307.34" y1="101.6" x2="307.34" y2="88.9" width="0.1524" layer="91"/>
+<wire x1="274.32" y1="104.14" x2="274.32" y2="109.22" width="0.1524" layer="91"/>
+<wire x1="274.32" y1="109.22" x2="287.02" y2="109.22" width="0.1524" layer="91"/>
 <pinref part="TP_ON/OFF" gate="G$1" pin="1"/>
 </segment>
@@
 <segment>
 <pinref part="U9" gate="G$1" pin="TRIM"/>
-<wire x1="302.26" y1="99.06" x2="304.8" y2="99.06" width="0.1524" layer="91"/>
-<wire x1="304.8" y1="99.06" x2="304.8" y2="83.82" width="0.1524" layer="91"/>
+<wire x1="276.86" y1="104.14" x2="276.86" y2="106.68" width="0.1524" layer="91"/>
+<wire x1="276.86" y1="106.68" x2="292.1" y2="106.68" width="0.1524" layer="91"/>
 <pinref part="TP_TRIM" gate="G$1" pin="1"/>
 </segment>
@@
 <description>Relays 1-2</description>
 <plain>
-<text x="119.38" y="170.18" size="1.778" layer="91">TVS Diode</text>
 </plain>
 <instances>
